Commit message: Add FT sensor changes WIP for proper xarm setup

File: xarm_description/urdf/xarm_device.urdf.xacro (robot description, xacro)
@@ -17,4 +17,5 @@
   <xacro:arg name="ros2_control_plugin" default="uf_robot_hardware/UFRobotSystemHardware"/>
   <xacro:arg name="ros2_control_params" default=""/>
+  <xacro:arg name="add_ft_sensor" default="false"/>
   <xacro:arg name="add_realsense_d435i" default="false"/>
   <xacro:arg name="add_d435i_links" default="true"/>
@@ -47,4 +48,5 @@
     ros2_control_plugin="$(arg ros2_control_plugin)" robot_type="$(arg robot_type)"
     load_gazebo_plugin="true" ros2_control_params="$(arg ros2_control_params)"
+    add_ft_sensor="$(arg add_ft_sensor)"
     add_realsense_d435i="$(arg add_realsense_d435i)"
     add_d435i_links="$(arg add_d435i_links)"

File: xarm_description/urdf/xarm_device_macro.xacro (robot description, xacro)
@@ -19,4 +19,5 @@
     ros2_control_params:=''
     load_gazebo_plugin:=false
+    add_ft_sensor:=false
     add_realsense_d435i:=false
     add_d435i_links:=true
@@ -201,4 +202,14 @@
       </xacro:unless>
     </xacro:unless>
+    <xacro:if value="${add_ft_sensor}">
+      <!-- (xarm) Load 6-axis force-torque sensor URDF -->
+      <xacro:include filename="$(find xarm_description)/urdf/ft_sensor/ft_sensor.urdf.xacro" />
+      <xacro:ft_sensor_urdf prefix="${prefix}" />
+      <joint name="${prefix}joint_ft_sensor" type="fixed">
+        <origin xyz="0 0 0.052" rpy="0 0 -1.5708" />
+        <parent link="${prefix}link${dof}" />
+        <child link="${prefix}link_ft_sensor" />
+      </joint>
+    </xacro:if>
     <xacro:if value="${add_realsense_d435i}">
       <!-- (xarm) Load RealSense D435i URDF -->
@@ -213,9 +224,18 @@
       <link name="${prefix}link_eef"/>
     </xacro:unless>
-    <joint name="${prefix}joint_eef" type="fixed">
-      <origin xyz="0 0 0" rpy="0 0 0" />
-      <parent link="${prefix}link${dof}" />
-      <child link="${prefix}link_eef" />
-    </joint>
+    <xacro:if value="${add_ft_sensor}">
+      <joint name="${prefix}joint_eef" type="fixed">
+        <origin xyz="0 0 0.008" rpy="0 0 1.5708" />
+        <parent link="${prefix}link_ft_sensor" />
+        <child link="${prefix}link_eef" />
+      </joint>
+    </xacro:if>
+    <xacro:unless value="${add_ft_sensor}">
+      <joint name="${prefix}joint_eef" type="fixed">
+        <origin xyz="0 0 0.008" rpy="0 0 0" />
+        <parent link="${prefix}link${dof}" />
+        <child link="${prefix}link_eef" />
+      </joint>
+    </xacro:unless>
     <xacro:if value="${add_gripper}">
       <xacro:if value="${robot_type == 'lite'}">
